File: a.brd (EAGLE design)
At the start: 50 x 42.2 mm, 31 parts, among them CON1 PINHEAD_1X04-2.54, CON2 PINHEAD_1X08-2.54, SW1 TACT_SWITCH-1-1825910-4, SW2 TACT_SWITCH-1-1825910-4, X3 PINHEAD_1X06-2-MALE, X4 PINHEAD_2X03-PTH-2.54

Commit message: preRelease minor fixes
Parts:
- added C5: 47u, rc:C1206
- C1: value 100u -> 47u; device rc:C2917 -> rc:C1206
- moved C1 1.13 mm to (18.1, 26.0), turned to 90 degrees
- moved C2 0.48 mm to (22.6, 30.3)
Connections:
- net GND: now also C1.P$1, C5.P$1; no longer C1.-
- net VDD_3V3: now also C1.P$2, C5.P$2; no longer C1.+
Routing:
- net VDD_3V3: track 95.7 -> 91.7 mm
