File: b.brd (EAGLE design)
At the start: 50 x 86.5 mm, 65 parts, among them CN1 CON-2P-DG500-5.08, CN2 CON-3P-DG500-5.08, CN3 CON-2P-DG500-5.08, CN4 CON-3P-DG500-5.08, CN5 CON-2P-DG500-5.08, Q1 BCR133, U2 TPS563200, U3 ISO3082, U4 B1212S-1WR3, U5 L78L05ACD13TR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

Commit message: preRelease minor fixes
Changed lines of the file:
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@@
 <layer number="14" name="Route14" color="22" fill="1" visible="no" active="no"/>
 <layer number="15" name="Route15" color="23" fill="1" visible="no" active="no"/>
-<layer number="16" name="Bottom" color="1" fill="1" visible="yes" active="yes"/>
-<layer number="17" name="Pads" color="2" fill="1" visible="yes" active="yes"/>
-<layer number="18" name="Vias" color="2" fill="1" visible="yes" active="yes"/>
+<layer number="16" name="Bottom" color="1" fill="1" visible="no" active="yes"/>
+<layer number="17" name="Pads" color="2" fill="1" visible="no" active="yes"/>
+<layer number="18" name="Vias" color="2" fill="1" visible="no" active="yes"/>
 <layer number="19" name="Unrouted" color="6" fill="1" visible="yes" active="yes"/>
 <layer number="20" name="Dimension" color="24" fill="1" visible="yes" active="yes"/>
@@
 <layer number="22" name="bPlace" color="7" fill="1" visible="yes" active="yes"/>
 <layer number="23" name="tOrigins" color="15" fill="1" visible="no" active="yes"/>
-<layer number="24" name="bOrigins" color="15" fill="1" visible="yes" active="yes"/>
+<layer number="24" name="bOrigins" color="15" fill="1" visible="no" active="yes"/>
 <layer number="25" name="tNames" color="7" fill="1" visible="no" active="yes"/>
 <layer number="26" name="bNames" color="7" fill="1" visible="yes" active="yes"/>
@@
 <layer number="148" name="mDocument" color="7" fill="1" visible="no" active="no"/>
 <layer number="149" name="mReference" color="7" fill="1" visible="no" active="no"/>
-<layer number="150" name="Notes" color="7" fill="1" visible="yes" active="yes"/>
+<layer number="150" name="Notes" color="7" fill="1" visible="no" active="yes"/>
 <layer number="151" name="HeatSink" color="7" fill="1" visible="yes" active="yes"/>
 <layer number="152" name="_bDocu" color="7" fill="1" visible="yes" active="yes"/>
@@
 </attributes>
 <variantdefs>
-<variantdef name="basic"/>
 </variantdefs>
 <classes>
@@
 </element>
 <element name="X2" library="pinhead" library_urn="urn:adsk.eagle:library:2540341" package="1X09-PTH-2.54" package3d_urn="urn:adsk.eagle:package:42601803/1" value="PINHEAD_1X09-2.54-TH-MALE" x="3.44" y="35.65" locked="yes" smashed="yes" rot="R270">
-<attribute name="NAME" x="5.44" y="35.65" locked="yes" size="1" layer="25" font="vector" ratio="15" rot="R270" align="center"/>
+<attribute name="NAME" x="1.14" y="35.65" size="1" layer="25" font="vector" ratio="15" rot="R270" align="center"/>
 </element>
 <element name="U$1" library="ref" package="REF_B" value="" x="0" y="0" smashed="yes"/>
@@
 <vertex x="27.5" y="0"/>
 </polygon>
-<wire x1="45.925" y1="21.175" x2="45.75" y2="21" width="0.5" layer="16"/>
 <via x="45.75" y="21" extent="1-16" drill="0.5" diameter="1"/>
 <via x="47" y="21" extent="1-16" drill="0.5" diameter="1"/>
